File: instromentataion yukseltec.kicad_sch (KiCad schematic)
At the start: 0 parts

Commit message: sil_emri
Other:
- note added: "merhaba benim ismim ahmedd kardes napyon soru sorma kardesim tamam kiral pardon sil sunu"
- note removed: "merhaba benim ismim ahmedd kardes napyon soru sorma kardesim tamam kiral pardon"
Changed lines of the file:
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@@
 	(generator_version "10.0")
 	(paper "A4")
-	(text "merhaba benim ismim ahmedd\nkardes napyon\nsoru sorma kardesim\ntamam kiral pardon"
+	(text "merhaba benim ismim ahmedd\nkardes napyon\nsoru sorma kardesim\ntamam kiral pardon\nsil sunu"
 		(exclude_from_sim no)
 		(at 139.7 95.25 0)
